File: Badge_v0.sch (EAGLE design)
At the start: 31 parts, among them U1 HX711, U2 ATMEGA328P_TQFP, U23 FT231X-Q, U3 BME680

Commit message: Initial routing, in progress
Parts:
- removed F1: PPTC1.5A, bschulz:PPTC1.5A
- removed R37: 330, bschulz_passives:R-EU_330R0402
- removed R63: 100k, bschulz_passives:R-EU_100KR0402
- added C1, C10, C11, C6: (no value), bschulz_passives:C-EU0.1UFC0603
- added C12: (no value), bschulz_passives:C-EU10UFC0805
- added C13, C14, C4, C9: (no value), bschulz_passives:C-EU1UFC0603
- added C2, C3: (no value), bschulz_passives:C-EUC0603
- added C5: (no value), bschulz_passives:C-EU0.1UFC0402
- added C7: 1uF, bschulz_passives:C-EU1UFC0603
- added C8: 300pF, bschulz_passives:C-EUC0603
- added D1, D2, D3, D5: LED0402, bschulz:LED0402
- added DS1: SAPRKFUN_MICRO_OLED, bschulz:SAPRKFUN_MICRO_OLED
- added H1, H2, H3, H4: (no value), bschulz:MOUNTING_HOLE4_PL
- added J3: CONN_82.54_SCREW, bschulz:CONN_82.54_SCREW
- added JP1: JUMPER-SMT_2_NC_PASTE_SILK, SparkFun-Jumpers:JUMPER-SMT_2_NC_PASTE_SILK
- added Q6: DMG3404, bschulz:MOSFET-NCH-DMG3404L
- added R1: 10k, bschulz_passives:R-EU_10KR0603
- added R2, R3: (no value), bschulz_passives:R-EU_10KR0603
- added R4: (no value), bschulz_passives:R-EU_P10KR0603
- added R5: (no value), bschulz_passives:R-EU_R0603
- added R6, R7, R8: (no value), bschulz_passives:R-EU_330R0402
- added S2: BUTTON, bschulz:BUTTON
- added U31: BME680, bschulz:BME680
- added U4: ISL29125, SparkFun-Sensors:ISL29125
- added U5: TPS7A0533DBV, bschulz:TPS7A0533DBV
- added XTAL1: CRYSTALHC-49/US, bschulz:CRYSTALHC-49/US
- D4: value CLVBA-FKA -> LED0402; device bschulz:CLVBA-FKA -> bschulz:LED0402
- MS1: value FEATHERWING -> FEATHERWINGLAYOUT; device adafruit:FEATHERWING -> bschulz:FEATHERWINGLAYOUT
- R38, R40: value 330 -> 1k
- R41: value 10k -> 100k
- U1: value HX711 -> MCP3421A3; device SparkFun-IC-Conversion:HX711 -> bschulz:MCP3421A3
- U3: value BME680 -> MCP15012.5V; device bschulz:BME680 -> bschulz:MCP15012.5V
Connections:
- removed net 3V3_AUX: C32.1, R41.2, RTC1.VCC, SD2.VDD
- removed net 3V3_CORE: D4.ANODE, ISP1.VCC
- removed net ALIVE_LED: R37.2
- removed net MOSI_BUF: SD2.DATA_IN
- removed net N$56: D4.GREEN_CATH, R37.1
- removed net RST: ISP1.RST
- removed net SCK_BUF: SD2.SCLK
- removed net SDA_OB: RTC1.SDA
- removed net SD_CS_BUF: SD2.CS
- removed net VUSB_POWER: F1.2, R63.2
- new net 3V3: C11.1, C12.1, C14.1, C32.1, C4.1, C6.1, C7.1, DS1.3V3, ISP1.VCC, J1.VCC, J3.2, R1.2, R2.2, R3.2, R41.2, R5.1, R6.2, R7.2, R8.2, RTC1.VCC, SD2.VDD, U1.VDD, U2.AVCC, U2.VCC@4, U2.VCC@6, U3.VDD, U31.CSB, U31.SDO, U31.VDD, U31.VDDIO, U5.VOUT
- new net AIN: J3.5, JP1.1, U1.VIN+
- new net IMU_INT: U2.PC0(ADC0), U4.!INT
- new net INT: J3.6, U2.PD3(INT1)
- new net JOY_DOWN: S1.DOWN, U2.PD5(T1)
- new net JOY_LEFT: S1.LEFT, U2.PC2(ADC2)
- new net JOY_PUSH: S1.CENT, U2.PC3(ADC3)
- new net JOY_RIGHT: S1.RIGHT, U2.PC1(ADC1)
- new net JOY_UP: S1.UP, U2.PD4(XCK/T0)
- new net LED_BLUE: D5.CATHODE, U2.PB2(SS/OC1B)
- new net LED_GREEN: D4.CATHODE, U2.PB1(OC1A)
- new net LED_RED: D3.CATHODE, U2.PD6(AIN0)
- new net N$10: D3.ANODE, R6.1
- new net N$11: D4.ANODE, R7.1
- new net N$12: D5.ANODE, R8.1
- new net N$2: JP1.2, R4.1
- new net N$3: C10.1, C9.1, R5.2, U4.VDD
- new net N$5: C1.1, U2.AREF
- new net N$7: C3.2, U2.PB7(XTAL2/TOSC2), XTAL1.1
- new net N$8: C2.2, U2.PB6(XTAL1/TOSC1), XTAL1.2
- new net REF_SHDN: U3.!SHDN
- new net RESET: C5.2, DS1.RST, ISP1.RST, MS1.!RESET, R1.1, S2.3, S2.4, U2.PC6(/RESET)
- new net SDA: DS1.D1, J1.SDA, J3.3, MS1.GPIOSDA, R2.1, RTC1.SDA, U1.SDA, U2.PC4(ADC4/SDA), U31.SDI, U4.SDA
- new net SD_CS: SD2.CS, U2.PB0(ICP)
- new net VIN+: C13.1, J2.+, MS1.VBAT, Q6.G, U5.EN, U5.VIN
- new net VIN-: J2.-, Q6.D
- new net VREF: C8.1, R4.2, U3.OUT
- net 3V3_FTDI: now also D1.ANODE, D2.ANODE
- net DTR: now also C5.1
- net GND: now also C1.2, C10.2, C11.2, C12.2, C13.2, C14.2, C2.1, C3.1, C4.2, C6.2, C7.2, C8.2, C9.2, DS1.D/C, DS1.GND, J1.GND, J3.1, MS1.GND, Q6.S, S1.GND, S2.1, S2.2, U1.VIN-, U1.VSS, U2.AGND, U2.GND@3, U2.GND@5, U3.GND, U31.GND, U4.GND, U5.GND; no longer R63.1
- net MISO: now also MS1.GPIOMISO, U2.PB4(MISO)
- net MOSI: now also MS1.GPIOMOSI, SD2.DATA_IN, U2.PB3(MOSI/OC2)
- net N$53: now also D2.CATHODE; no longer D4.RED_CATH
- net N$54: now also D1.CATHODE; no longer D4.BLUE_CATH
- net RTC_INT: now also U2.PD2(INT0)
- net RX: now also J3.8, MS1.GPIOTX, U2.PD0(RXD)
- net SCK: now also MS1.GPIOSCK, SD2.SCLK, U2.PB5(SCK)
- net SCL: now also DS1.D0, J1.SCL, J3.4, MS1.GPIOSCL, R3.1, U1.SCL, U2.PC5(ADC5/SCL), U31.SCK, U4.SCL
- net SD_CD: now also U2.PD7(AIN1)
- net TX: now also J3.7, MS1.GPIORX, U2.PD1(TXD)
- net VUSB: no longer F1.1
Other:
- note added: "flex"
